Commit message: removed build install log files in src

File: ros2_ws/src/robotiq_3f_gripper_description/urdf/robotiq_3f_gripper_ros2_control.xacro (robot description, xacro)
@@ -1,12 +1,7 @@
 <?xml version="1.0"?>
-<!--
-robotiq_3f_gripper_ros2_control(prefix, sim_ignition)
-Exposes only the 3 base knuckle joints (one per finger) as actuated
-DOFs to ros2_control. joint_2/joint_3 per finger remain fixed (see
-robotiq_3f_finger_macro.xacro) -- this is a deliberate simplification
-for a first working gripper-in-the-loop simulation.
--->
 <robot xmlns:xacro="http://ros.org/wiki/xacro">
-  <xacro:macro name="robotiq_3f_gripper_ros2_control" params="prefix sim_ignition:=true">
+  <xacro:macro
+    name="robotiq_3f_gripper_ros2_control"
+    params="prefix sim_ignition:=true">
     <ros2_control name="${prefix}gripper_system" type="system">
       <hardware>
