Commit message: Restore Robotiq middle-finger mirrored geometry
Co-authored-by: Copilot <223556219+Copilot@users.noreply.github.com>

File: ros2_ws/src/robotiq_3f_gripper_description/urdf/robotiq_3f_finger_macro.xacro (robot description, xacro)
@@ -7,5 +7,5 @@
 -->
 <robot xmlns:xacro="http://ros.org/wiki/xacro">
-  <xacro:macro name="robotiq_3f_finger_articulated" params="prefix">
+  <xacro:macro name="robotiq_3f_finger_articulated" params="prefix axis_sign=1">
     <link name="${prefix}link_0">
       <visual>
@@ -95,8 +95,8 @@
       <parent link="${prefix}link_0"/>
       <child link="${prefix}link_1"/>
-      <!-- Keep the finger axis aligned with the official Robotiq Z-axis rotation.
-           This is not mirrored or flipped relative to the palm frame, and the
-           commanded position stays in the valid positive range. -->
-      <axis xyz="0 0 1"/>
+      <!-- Keep the side-finger axis aligned to the official Robotiq Z-axis rotation.
+           The middle finger uses a dedicated mirrored macro below so the center
+           finger matches the physical Robotiq layout without a flipped command set. -->
+      <axis xyz="0 0 ${axis_sign}"/>
       <origin xyz="0.020 0 0" rpy="0 0 0"/>
       <limit lower="0.0495" upper="1.2218" effort="100" velocity="1.0"/>
@@ -113,3 +113,108 @@
     </joint>
   </xacro:macro>
+  <xacro:macro name="robotiq_3f_middle_finger_articulated" params="prefix">
+    <link name="${prefix}link_0">
+      <visual>
+        <origin xyz="0.020 0 0" rpy="0 0 0"/>
+        <geometry>
+          <mesh filename="package://robotiq_3f_gripper_description/meshes/visual/link_0.dae"/>
+        </geometry>
+        <material name="gripper_dark">
+          <color rgba="0.12 0.12 0.13 1"/>
+        </material>
+      </visual>
+      <collision>
+        <origin xyz="0.020 0 0" rpy="0 0 0"/>
+        <geometry>
+          <mesh filename="package://robotiq_3f_gripper_description/meshes/collision/link_0.STL"/>
+        </geometry>
+      </collision>
+      <inertial>
+          <origin xyz="0 0 0" rpy="0 0 0"/>
+          <mass value="0.05"/>
+          <inertia ixx="4.9e-6" ixy="0" ixz="0" iyy="9.1e-6" iyz="0" izz="9.1e-6" />
+      </inertial>
+    </link>
+    <link name="${prefix}link_1">
+      <visual>
+        <origin xyz="0.050 0.028 0" rpy="0 0 0.52"/>
+        <geometry>
+          <mesh filename="package://robotiq_3f_gripper_description/meshes/visual/link_1.dae"/>
+        </geometry>
+        <material name="gripper_light">
+          <color rgba="0.65 0.66 0.68 1"/>
+        </material>
+      </visual>
+      <collision>
+        <origin xyz="0.050 0.028 0" rpy="0 0 0.52"/>
+        <geometry>
+          <mesh filename="package://robotiq_3f_gripper_description/meshes/collision/link_1.STL"/>
+        </geometry>
+      </collision>
+      <inertial>
+          <origin xyz="0 0 0" rpy="0 0 0"/>
+          <mass value="0.15"/>
+          <inertia ixx="1.08e-5" ixy="0" ixz="0" iyy="6.67e-5" iyz="0" izz="6.67e-5" />
+      </inertial>
+    </link>
+    <link name="${prefix}link_2">
+      <visual>
+        <origin xyz="0.039 0 0.0075" rpy="0 0 0"/>
+        <geometry>
+          <mesh filename="package://robotiq_3f_gripper_description/meshes/visual/link_2.dae"/>
+        </geometry>
+        <material name="gripper_light"/>
+      </visual>
+      <collision>
+        <origin xyz="0.039 0 0.0075" rpy="0 0 0"/>
+        <geometry>
+          <mesh filename="package://robotiq_3f_gripper_description/meshes/collision/link_2.STL"/>
+        </geometry>
+      </collision>
+      <inertial>
+          <origin xyz="0 0 0" rpy="0 0 0"/>
+          <mass value="0.05"/>
+          <inertia ixx="2.5e-6" ixy="0" ixz="0" iyy="7.9e-6" iyz="0" izz="7.9e-6" />
+      </inertial>
+    </link>
+    <link name="${prefix}link_3">
+      <visual>
+        <origin xyz="0 0 0" rpy="0 0 -0.52"/>
+        <geometry>
+          <mesh filename="package://robotiq_3f_gripper_description/meshes/visual/link_3.dae"/>
+        </geometry>
+        <material name="gripper_light"/>
+      </visual>
+      <collision>
+        <origin xyz="0 0 0" rpy="0 0 -0.52"/>
+        <geometry>
+          <mesh filename="package://robotiq_3f_gripper_description/meshes/collision/link_3.STL"/>
+        </geometry>
+      </collision>
+      <inertial>
+        <origin xyz="0 0 0" rpy="0 0 0"/>
+        <mass value="0.05"/>
+        <inertia ixx="0.001239" ixy="-0.000251" ixz="0.000019" iyy="0.00085" iyz="0" izz="0.001632"/>
+      </inertial>
+    </link>
+    <joint name="${prefix}joint_1" type="revolute">
+      <parent link="${prefix}link_0"/>
+      <child link="${prefix}link_1"/>
+      <!-- The middle finger is mounted on the opposite side of the palm, so it
+           needs the mirrored sign to keep the physical closing motion consistent. -->
+      <axis xyz="0 0 -1"/>
+      <origin xyz="0.020 0 0" rpy="0 0 0"/>
+      <limit lower="0.0495" upper="1.2218" effort="100" velocity="1.0"/>
+    </joint>
+    <joint name="${prefix}joint_2" type="fixed">
+      <parent link="${prefix}link_1"/>
+      <child link="${prefix}link_2"/>
+      <origin xyz="0.050 0.028 0" rpy="0 0 0.52"/>
+    </joint>
+    <joint name="${prefix}joint_3" type="fixed">
+      <parent link="${prefix}link_2"/>
+      <child link="${prefix}link_3"/>
+      <origin xyz="0.039 0 0" rpy="0 0 0"/>
+    </joint>
+  </xacro:macro>
 </robot>

File: ros2_ws/src/robotiq_3f_gripper_description/urdf/robotiq_3f_gripper_macro.xacro (robot description, xacro)
@@ -51,7 +51,7 @@
       <origin xyz="0.0 0.0875 0.0" rpy="0 0 1.5707"/>
     </joint>
-    <xacro:robotiq_3f_finger_articulated prefix="${prefix}finger_1_"/>
-    <xacro:robotiq_3f_finger_articulated prefix="${prefix}finger_2_"/>
-    <xacro:robotiq_3f_finger_articulated prefix="${prefix}finger_middle_"/>
+    <xacro:robotiq_3f_finger_articulated prefix="${prefix}finger_1_" axis_sign="1"/>
+    <xacro:robotiq_3f_finger_articulated prefix="${prefix}finger_2_" axis_sign="1"/>
+    <xacro:robotiq_3f_middle_finger_articulated prefix="${prefix}finger_middle_"/>
     <joint name="${prefix}palm_finger_1_joint" type="fixed">
       <parent link="${prefix}palm"/>
@@ -67,9 +67,8 @@
       <parent link="${prefix}palm"/>
       <child link="${prefix}finger_middle_link_0"/>
-      <!-- Preserve the official Robotiq 3F palm mount for the middle finger. The
-           frame is only yawed into the palm coordinate frame; no mirrored or flipped
-           axis is introduced, and the commanded joint values stay within the
-           positive URDF range defined in robotiq_3f_gripper_ros2_control.xacro. -->
-      <origin xyz="0.0455 0.0214 0" rpy="0 0 1.57"/>
+      <!-- The middle finger sits on the opposite side of the palm and needs the
+           same mirror/pitch adjustment that the original Robotiq geometry used,
+           while the mirrored joint sign keeps the command convention consistent. -->
+      <origin xyz="0.0455 0.0214 0" rpy="0 3.1416 1.57"/>
     </joint>
   </xacro:macro>
