Commit message: created moveit package for gripper movement

File: ros2_ws/src/robotiq_3f_gripper_description/urdf/robotiq_3f_finger_macro.xacro (robot description, xacro)
@@ -99,17 +99,13 @@
       <limit lower="0.0495" upper="1.2218" effort="100" velocity="1.0"/>
     </joint>
-    <joint name="${prefix}joint_2" type="revolute">
+    <joint name="${prefix}joint_2" type="fixed">
       <parent link="${prefix}link_1"/>
       <child link="${prefix}link_2"/>
-      <axis xyz="0 0 1"/>
       <origin xyz="0.050 -0.028 0" rpy="0 0 -0.52"/>
-      <limit lower="0.0" upper="1.5708" effort="100" velocity="1.0"/>
     </joint>
-    <joint name="${prefix}joint_3" type="revolute">
+    <joint name="${prefix}joint_3" type="fixed">
       <parent link="${prefix}link_2"/>
       <child link="${prefix}link_3"/>
-      <axis xyz="0 0 1"/>
       <origin xyz="0.039 0 0" rpy="0 0 0"/>
-      <limit lower="-1.2217" upper="-0.0523" effort="100" velocity="1.0"/>
     </joint>
   </xacro:macro>

File: ros2_ws/src/robotiq_3f_gripper_description/urdf/robotiq_3f_gripper_macro.xacro (robot description, xacro)
@@ -50,17 +50,13 @@
     <xacro:robotiq_3f_finger_articulated prefix="${prefix}finger_2_"/>
     <xacro:robotiq_3f_finger_articulated prefix="${prefix}finger_middle_"/>
-    <joint name="${prefix}palm_finger_1_joint" type="revolute">
+    <joint name="${prefix}palm_finger_1_joint" type="fixed">
       <parent link="${prefix}palm"/>
       <child link="${prefix}finger_1_link_0"/>
-      <axis xyz="0 1 0"/>
       <origin xyz="-0.0455 0.0214 0.036" rpy="0 3.1416 -1.57"/>
-      <limit lower="-0.1784" upper="0.192" effort="100" velocity="1.0"/>
     </joint>
-    <joint name="${prefix}palm_finger_2_joint" type="revolute">
+    <joint name="${prefix}palm_finger_2_joint" type="fixed">
       <parent link="${prefix}palm"/>
       <child link="${prefix}finger_2_link_0"/>
-      <axis xyz="0 1 0"/>
       <origin xyz="-0.0455 0.0214 -0.036" rpy="0 3.1416 -1.57"/>
-      <limit lower="-0.192" upper="0.1784" effort="100" velocity="1.0"/>
     </joint>
     <joint name="${prefix}palm_finger_middle_joint" type="fixed">

File: ros2_ws/src/robotiq_3f_gripper_description/urdf/ur10_robotiq_3f.urdf.xacro (robot description, xacro)
@@ -1,48 +1,14 @@
 <?xml version="1.0"?>
-<!--
-ur10_robotiq_3f.urdf.xacro
-Combines the stock Universal_Robots_ROS2_Description UR10 arm with the
-ported Robotiq 3-Finger Adaptive Gripper (articulated), attached at the
-arm's "tool0" link.
-This purposefully does NOT modify ur_description's files. It only
-includes ur_macro.xacro (as ur.urdf.xacro does) and adds the gripper
-on top, so upstream UR description updates can still be pulled cleanly.
--->
 <robot xmlns:xacro="http://wiki.ros.org/xacro" name="$(arg name)">
-  <xacro:arg name="name" default="ur"/>
-  <xacro:include filename="$(find ur_description)/urdf/ur_macro.xacro"/>
+  <xacro:arg name="name" default="ur10"/>
+  <xacro:arg name="tf_prefix" default=""/>
+  <xacro:arg name="gripper_prefix" default="gripper_"/>
+  <xacro:arg name="sim_ignition" default="true"/>
+  <xacro:include filename="$(find ur_description)/urdf/ur.urdf.xacro"/>
   <xacro:include filename="$(find robotiq_3f_gripper_description)/urdf/robotiq_3f_gripper_macro.xacro"/>
-  <!-- possible 'ur_type' values: ur3, ur5, ur10, ur3e, ur5e, ur7e, ur10e, ur12e, ur16e, ur8long, ur15, ur18, ur20, ur30 -->
-  <xacro:arg name="ur_type" default="ur10"/>
-  <xacro:arg name="tf_prefix" default=""/>
-  <xacro:arg name="joint_limit_params" default="$(find ur_description)/config/$(arg ur_type)/joint_limits.yaml"/>
-  <xacro:arg name="kinematics_params" default="$(find ur_description)/config/$(arg ur_type)/default_kinematics.yaml"/>
-  <xacro:arg name="physical_params" default="$(find ur_description)/config/$(arg ur_type)/physical_parameters.yaml"/>
-  <xacro:arg name="visual_params" default="$(find ur_description)/config/$(arg ur_type)/visual_parameters.yaml"/>
-  <xacro:arg name="transmission_hw_interface" default=""/>
-  <xacro:arg name="safety_limits" default="false"/>
-  <xacro:arg name="safety_pos_margin" default="0.15"/>
-  <xacro:arg name="safety_k_position" default="20"/>
-  <!-- gripper prefix, in case you ever need two arms/grippers in one urdf -->
-  <xacro:arg name="gripper_prefix" default="gripper_"/>
-  <link name="world"/>
-  <xacro:ur_robot
-    name="$(arg name)"
-    tf_prefix="$(arg tf_prefix)"
-    parent="world"
-    joint_limits_parameters_file="$(arg joint_limit_params)"
-    kinematics_parameters_file="$(arg kinematics_params)"
-    physical_parameters_file="$(arg physical_params)"
-    visual_parameters_file="$(arg visual_params)"
-    safety_limits="$(arg safety_limits)"
-    safety_pos_margin="$(arg safety_pos_margin)"
-    safety_k_position="$(arg safety_k_position)"
-    >
-    <origin xyz="0 0 0" rpy="0 0 0"/>
-  </xacro:ur_robot>
-  <!-- attach the 3-finger gripper to the arm's tool0.
-       tf_prefix (if you set one) is applied to tool0 too. -->
-    <xacro:robotiq_3f_gripper_articulated prefix="$(arg gripper_prefix)" parent="$(arg tf_prefix)tool0">
-      <origin xyz="0 0 0" rpy="1.5708 0 0"/>
-    </xacro:robotiq_3f_gripper_articulated>
+  <xacro:include filename="$(find robotiq_3f_gripper_description)/urdf/robotiq_3f_gripper_ros2_control.xacro"/>
+  <xacro:robotiq_3f_gripper_articulated prefix="$(arg gripper_prefix)" parent="$(arg tf_prefix)tool0">
+    <origin xyz="0 0 0" rpy="1.5708 0 0"/>
+  </xacro:robotiq_3f_gripper_articulated>
+  <xacro:robotiq_3f_gripper_ros2_control prefix="$(arg gripper_prefix)" sim_ignition="$(arg sim_ignition)"/>
 </robot>

Commit message: Refactor gripper macros to include axis_sign for consistent finger motion and update gripper_test.py comments for clarity

File: ros2_ws/src/robotiq_3f_gripper_description/urdf/robotiq_3f_finger_macro.xacro (robot description, xacro)
@@ -7,5 +7,5 @@
 -->
 <robot xmlns:xacro="http://ros.org/wiki/xacro">
-  <xacro:macro name="robotiq_3f_finger_articulated" params="prefix">
+  <xacro:macro name="robotiq_3f_finger_articulated" params="prefix axis_sign=1">
     <link name="${prefix}link_0">
       <visual>
@@ -95,5 +95,5 @@
       <parent link="${prefix}link_0"/>
       <child link="${prefix}link_1"/>
-      <axis xyz="0 0 1"/>
+      <axis xyz="0 0 ${axis_sign}"/>
       <origin xyz="0.020 0 0" rpy="0 0 0"/>
       <limit lower="0.0495" upper="1.2218" effort="100" velocity="1.0"/>
@@ -110,3 +110,108 @@
     </joint>
   </xacro:macro>
+  <xacro:macro name="robotiq_3f_middle_finger_articulated" params="prefix">
+    <link name="${prefix}link_0">
+      <visual>
+        <origin xyz="0.020 0 0" rpy="0 0 0"/>
+        <geometry>
+          <mesh filename="package://robotiq_3f_gripper_description/meshes/visual/link_0.dae"/>
+        </geometry>
+        <material name="gripper_dark">
+          <color rgba="0.12 0.12 0.13 1"/>
+        </material>
+      </visual>
+      <collision>
+        <origin xyz="0.020 0 0" rpy="0 0 0"/>
+        <geometry>
+          <mesh filename="package://robotiq_3f_gripper_description/meshes/collision/link_0.STL"/>
+        </geometry>
+      </collision>
+      <inertial>
+          <origin xyz="0 0 0" rpy="0 0 0"/>
+          <mass value="0.05"/>
+          <inertia ixx="4.9e-6" ixy="0" ixz="0" iyy="9.1e-6" iyz="0" izz="9.1e-6" />
+      </inertial>
+    </link>
+    <link name="${prefix}link_1">
+      <visual>
+        <origin xyz="0.050 0.028 0" rpy="0 0 0.52"/>
+        <geometry>
+          <mesh filename="package://robotiq_3f_gripper_description/meshes/visual/link_1.dae"/>
+        </geometry>
+        <material name="gripper_light">
+          <color rgba="0.65 0.66 0.68 1"/>
+        </material>
+      </visual>
+      <collision>
+        <origin xyz="0.050 0.028 0" rpy="0 0 0.52"/>
+        <geometry>
+          <mesh filename="package://robotiq_3f_gripper_description/meshes/collision/link_1.STL"/>
+        </geometry>
+      </collision>
+      <inertial>
+          <origin xyz="0 0 0" rpy="0 0 0"/>
+          <mass value="0.15"/>
+          <inertia ixx="1.08e-5" ixy="0" ixz="0" iyy="6.67e-5" iyz="0" izz="6.67e-5" />
+      </inertial>
+    </link>
+    <link name="${prefix}link_2">
+      <visual>
+        <origin xyz="0.039 0 0.0075" rpy="0 0 0"/>
+        <geometry>
+          <mesh filename="package://robotiq_3f_gripper_description/meshes/visual/link_2.dae"/>
+        </geometry>
+        <material name="gripper_light"/>
+      </visual>
+      <collision>
+        <origin xyz="0.039 0 0.0075" rpy="0 0 0"/>
+        <geometry>
+          <mesh filename="package://robotiq_3f_gripper_description/meshes/collision/link_2.STL"/>
+        </geometry>
+      </collision>
+      <inertial>
+          <origin xyz="0 0 0" rpy="0 0 0"/>
+          <mass value="0.05"/>
+          <inertia ixx="2.5e-6" ixy="0" ixz="0" iyy="7.9e-6" iyz="0" izz="7.9e-6" />
+      </inertial>
+    </link>
+    <link name="${prefix}link_3">
+      <visual>
+        <origin xyz="0 0 0" rpy="0 0 -0.52"/>
+        <geometry>
+          <mesh filename="package://robotiq_3f_gripper_description/meshes/visual/link_3.dae"/>
+        </geometry>
+        <material name="gripper_light"/>
+      </visual>
+      <collision>
+        <origin xyz="0 0 0" rpy="0 0 -0.52"/>
+        <geometry>
+          <mesh filename="package://robotiq_3f_gripper_description/meshes/collision/link_3.STL"/>
+        </geometry>
+      </collision>
+      <inertial>
+        <origin xyz="0 0 0" rpy="0 0 0"/>
+        <mass value="0.05"/>
+        <inertia ixx="0.001239" ixy="-0.000251" ixz="0.000019" iyy="0.00085" iyz="0" izz="0.001632"/>
+      </inertial>
+    </link>
+    <joint name="${prefix}joint_1" type="revolute">
+      <parent link="${prefix}link_0"/>
+      <child link="${prefix}link_1"/>
+      <!-- Keep the middle finger mirrored to the side fingers while preserving a
+           consistent positive-closing convention for the controller. -->
+      <axis xyz="0 0 -1"/>
+      <origin xyz="0.020 0 0" rpy="0 0 0"/>
+      <limit lower="0.0495" upper="1.2218" effort="100" velocity="1.0"/>
+    </joint>
+    <joint name="${prefix}joint_2" type="fixed">
+      <parent link="${prefix}link_1"/>
+      <child link="${prefix}link_2"/>
+      <origin xyz="0.050 0.028 0" rpy="0 0 0.52"/>
+    </joint>
+    <joint name="${prefix}joint_3" type="fixed">
+      <parent link="${prefix}link_2"/>
+      <child link="${prefix}link_3"/>
+      <origin xyz="0.039 0 0" rpy="0 0 0"/>
+    </joint>
+  </xacro:macro>
 </robot>

File: ros2_ws/src/robotiq_3f_gripper_description/urdf/robotiq_3f_gripper_macro.xacro (robot description, xacro)
@@ -51,22 +51,10 @@
       <origin xyz="0.0 0.0875 0.0" rpy="0 0 1.5707"/>
     </joint>
-    <xacro:robotiq_3f_finger_articulated prefix="${prefix}finger_1_"/>
-    <xacro:robotiq_3f_finger_articulated prefix="${prefix}finger_2_"/>
-    <xacro:robotiq_3f_finger_articulated prefix="${prefix}finger_middle_"/>
-    <gazebo reference="${prefix}palm">
-      <selfCollide>false</selfCollide>
-    </gazebo>
-    <gazebo reference="${prefix}finger_middle_link_0">
-      <selfCollide>false</selfCollide>
-    </gazebo>
-    <gazebo reference="${prefix}finger_middle_link_1">
-      <selfCollide>false</selfCollide>
-    </gazebo>
-    <gazebo reference="${prefix}finger_middle_link_2">
-      <selfCollide>false</selfCollide>
-    </gazebo>
-    <gazebo reference="${prefix}finger_middle_link_3">
-      <selfCollide>false</selfCollide>
-    </gazebo>
+    <!-- The middle finger's axis is intentionally inverted so that the same positive
+         command signals all three fingers to close/open in the same physical direction.
+         Keep the palm mount orientation at 0 0 1.57 to preserve the Robotiq layout. -->
+    <xacro:robotiq_3f_finger_articulated prefix="${prefix}finger_1_" axis_sign="1"/>
+    <xacro:robotiq_3f_finger_articulated prefix="${prefix}finger_2_" axis_sign="1"/>
+    <xacro:robotiq_3f_middle_finger_articulated prefix="${prefix}finger_middle_"/>
     <joint name="${prefix}palm_finger_1_joint" type="fixed">
       <parent link="${prefix}palm"/>
@@ -82,5 +70,8 @@
       <parent link="${prefix}palm"/>
       <child link="${prefix}finger_middle_link_0"/>
-      <origin xyz="0.0455 0.0214 0" rpy="0 0 1.57"/>
+      <!-- The middle finger is mounted on the opposite side of the palm, so it needs the
+           same 180° pitch flip as the mirrored A/B finger frames. This keeps the center
+           finger facing the other two instead of lying in the same in-plane orientation. -->
+      <origin xyz="0.0455 0.0214 0" rpy="0 3.1416 1.57"/>
     </joint>
   </xacro:macro>

Commit message: Refactor gripper macros for consistency and update collision handling in URDF/SRDF configurations

File: ros2_ws/src/robotiq_3f_gripper_description/urdf/robotiq_3f_finger_macro.xacro (robot description, xacro)
@@ -110,108 +110,3 @@
     </joint>
   </xacro:macro>
-  <xacro:macro name="robotiq_3f_middle_finger_articulated" params="prefix">
-    <link name="${prefix}link_0">
-      <visual>
-        <origin xyz="0.020 0 0" rpy="0 0 0"/>
-        <geometry>
-          <mesh filename="package://robotiq_3f_gripper_description/meshes/visual/link_0.dae"/>
-        </geometry>
-        <material name="gripper_dark">
-          <color rgba="0.12 0.12 0.13 1"/>
-        </material>
-      </visual>
-      <collision>
-        <origin xyz="0.020 0 0" rpy="0 0 0"/>
-        <geometry>
-          <mesh filename="package://robotiq_3f_gripper_description/meshes/collision/link_0.STL"/>
-        </geometry>
-      </collision>
-      <inertial>
-          <origin xyz="0 0 0" rpy="0 0 0"/>
-          <mass value="0.05"/>
-          <inertia ixx="4.9e-6" ixy="0" ixz="0" iyy="9.1e-6" iyz="0" izz="9.1e-6" />
-      </inertial>
-    </link>
-    <link name="${prefix}link_1">
-      <visual>
-        <origin xyz="0.050 0.028 0" rpy="0 0 0.52"/>
-        <geometry>
-          <mesh filename="package://robotiq_3f_gripper_description/meshes/visual/link_1.dae"/>
-        </geometry>
-        <material name="gripper_light">
-          <color rgba="0.65 0.66 0.68 1"/>
-        </material>
-      </visual>
-      <collision>
-        <origin xyz="0.050 0.028 0" rpy="0 0 0.52"/>
-        <geometry>
-          <mesh filename="package://robotiq_3f_gripper_description/meshes/collision/link_1.STL"/>
-        </geometry>
-      </collision>
-      <inertial>
-          <origin xyz="0 0 0" rpy="0 0 0"/>
-          <mass value="0.15"/>
-          <inertia ixx="1.08e-5" ixy="0" ixz="0" iyy="6.67e-5" iyz="0" izz="6.67e-5" />
-      </inertial>
-    </link>
-    <link name="${prefix}link_2">
-      <visual>
-        <origin xyz="0.039 0 0.0075" rpy="0 0 0"/>
-        <geometry>
-          <mesh filename="package://robotiq_3f_gripper_description/meshes/visual/link_2.dae"/>
-        </geometry>
-        <material name="gripper_light"/>
-      </visual>
-      <collision>
-        <origin xyz="0.039 0 0.0075" rpy="0 0 0"/>
-        <geometry>
-          <mesh filename="package://robotiq_3f_gripper_description/meshes/collision/link_2.STL"/>
-        </geometry>
-      </collision>
-      <inertial>
-          <origin xyz="0 0 0" rpy="0 0 0"/>
-          <mass value="0.05"/>
-          <inertia ixx="2.5e-6" ixy="0" ixz="0" iyy="7.9e-6" iyz="0" izz="7.9e-6" />
-      </inertial>
-    </link>
-    <link name="${prefix}link_3">
-      <visual>
-        <origin xyz="0 0 0" rpy="0 0 -0.52"/>
-        <geometry>
-          <mesh filename="package://robotiq_3f_gripper_description/meshes/visual/link_3.dae"/>
-        </geometry>
-        <material name="gripper_light"/>
-      </visual>
-      <collision>
-        <origin xyz="0 0 0" rpy="0 0 -0.52"/>
-        <geometry>
-          <mesh filename="package://robotiq_3f_gripper_description/meshes/collision/link_3.STL"/>
-        </geometry>
-      </collision>
-      <inertial>
-        <origin xyz="0 0 0" rpy="0 0 0"/>
-        <mass value="0.05"/>
-        <inertia ixx="0.001239" ixy="-0.000251" ixz="0.000019" iyy="0.00085" iyz="0" izz="0.001632"/>
-      </inertial>
-    </link>
-    <joint name="${prefix}joint_1" type="revolute">
-      <parent link="${prefix}link_0"/>
-      <child link="${prefix}link_1"/>
-      <!-- Keep the middle finger mirrored to the side fingers while preserving a
-           consistent positive-closing convention for the controller. -->
-      <axis xyz="0 0 -1"/>
-      <origin xyz="0.020 0 0" rpy="0 0 0"/>
-      <limit lower="0.0495" upper="1.2218" effort="100" velocity="1.0"/>
-    </joint>
-    <joint name="${prefix}joint_2" type="fixed">
-      <parent link="${prefix}link_1"/>
-      <child link="${prefix}link_2"/>
-      <origin xyz="0.050 0.028 0" rpy="0 0 0.52"/>
-    </joint>
-    <joint name="${prefix}joint_3" type="fixed">
-      <parent link="${prefix}link_2"/>
-      <child link="${prefix}link_3"/>
-      <origin xyz="0.039 0 0" rpy="0 0 0"/>
-    </joint>
-  </xacro:macro>
 </robot>

File: ros2_ws/src/robotiq_3f_gripper_description/urdf/robotiq_3f_gripper_macro.xacro (robot description, xacro)
@@ -56,5 +56,5 @@
     <xacro:robotiq_3f_finger_articulated prefix="${prefix}finger_1_" axis_sign="1"/>
     <xacro:robotiq_3f_finger_articulated prefix="${prefix}finger_2_" axis_sign="1"/>
-    <xacro:robotiq_3f_middle_finger_articulated prefix="${prefix}finger_middle_"/>
+    <xacro:robotiq_3f_finger_articulated prefix="${prefix}finger_middle_" axis_sign="1"/>
     <joint name="${prefix}palm_finger_1_joint" type="fixed">
       <parent link="${prefix}palm"/>
@@ -73,5 +73,5 @@
            same 180° pitch flip as the mirrored A/B finger frames. This keeps the center
            finger facing the other two instead of lying in the same in-plane orientation. -->
-      <origin xyz="0.0455 0.0214 0" rpy="0 3.1416 1.57"/>
+      <origin xyz="0.0455 0.0214 0" rpy="0 0 1.57"/>
     </joint>
   </xacro:macro>

File: ros2_ws/src/robotiq_3f_gripper_description/urdf/robotiq_3f_gripper_ros2_control.xacro (robot description, xacro)
@@ -14,16 +14,31 @@
       </hardware>
       <joint name="${prefix}finger_1_joint_1">
-        <command_interface name="position"/>
-        <state_interface name="position"/>
+        <command_interface name="position">
+          <param name="min">0.0495</param>
+          <param name="max">1.2218</param>
+        </command_interface>
+        <state_interface name="position">
+          <param name="initial_value">0.0495</param>
+        </state_interface>
         <state_interface name="velocity"/>
       </joint>
       <joint name="${prefix}finger_2_joint_1">
-        <command_interface name="position"/>
-        <state_interface name="position"/>
+        <command_interface name="position">
+          <param name="min">0.0495</param>
+          <param name="max">1.2218</param>
+        </command_interface>
+        <state_interface name="position">
+          <param name="initial_value">0.0495</param>
+        </state_interface>
         <state_interface name="velocity"/>
       </joint>
       <joint name="${prefix}finger_middle_joint_1">
-        <command_interface name="position"/>
-        <state_interface name="position"/>
+        <command_interface name="position">
+          <param name="min">0.0495</param>
+          <param name="max">1.2218</param>
+        </command_interface>
+        <state_interface name="position">
+          <param name="initial_value">0.0495</param>
+        </state_interface>
         <state_interface name="velocity"/>
       </joint>

Commit message: not working - debugging steps

File: ros2_ws/src/robotiq_3f_gripper_description/urdf/robotiq_3f_finger_macro.xacro (robot description, xacro)
@@ -7,5 +7,5 @@
 -->
 <robot xmlns:xacro="http://ros.org/wiki/xacro">
-  <xacro:macro name="robotiq_3f_finger_articulated" params="prefix axis_sign=1">
+  <xacro:macro name="robotiq_3f_finger_articulated" params="prefix">
     <link name="${prefix}link_0">
       <visual>
@@ -95,5 +95,5 @@
       <parent link="${prefix}link_0"/>
       <child link="${prefix}link_1"/>
-      <axis xyz="0 0 ${axis_sign}"/>
+      <axis xyz="0 0 1"/>
       <origin xyz="0.020 0 0" rpy="0 0 0"/>
       <limit lower="0.0495" upper="1.2218" effort="100" velocity="1.0"/>

File: ros2_ws/src/robotiq_3f_gripper_description/urdf/robotiq_3f_gripper_macro.xacro (robot description, xacro)
@@ -51,10 +51,7 @@
       <origin xyz="0.0 0.0875 0.0" rpy="0 0 1.5707"/>
     </joint>
-    <!-- The middle finger's axis is intentionally inverted so that the same positive
-         command signals all three fingers to close/open in the same physical direction.
-         Keep the palm mount orientation at 0 0 1.57 to preserve the Robotiq layout. -->
-    <xacro:robotiq_3f_finger_articulated prefix="${prefix}finger_1_" axis_sign="1"/>
-    <xacro:robotiq_3f_finger_articulated prefix="${prefix}finger_2_" axis_sign="1"/>
-    <xacro:robotiq_3f_finger_articulated prefix="${prefix}finger_middle_" axis_sign="1"/>
+    <xacro:robotiq_3f_finger_articulated prefix="${prefix}finger_1_"/>
+    <xacro:robotiq_3f_finger_articulated prefix="${prefix}finger_2_"/>
+    <xacro:robotiq_3f_finger_articulated prefix="${prefix}finger_middle_"/>
     <joint name="${prefix}palm_finger_1_joint" type="fixed">
       <parent link="${prefix}palm"/>
@@ -70,7 +67,7 @@
       <parent link="${prefix}palm"/>
       <child link="${prefix}finger_middle_link_0"/>
-      <!-- The middle finger is mounted on the opposite side of the palm, so it needs the
-           same 180° pitch flip as the mirrored A/B finger frames. This keeps the center
-           finger facing the other two instead of lying in the same in-plane orientation. -->
+      <!-- Official Robotiq 3F mounting: the middle finger is mounted with a yaw-only
+           rotation in the palm frame. The inverse motion is handled by the command-space
+           sign, not by rotating the physical frame away from the real Robotiq layout. -->
       <origin xyz="0.0455 0.0214 0" rpy="0 0 1.57"/>
     </joint>

File: ros2_ws/src/robotiq_3f_gripper_description/urdf/ur10_robotiq_3f.urdf.xacro (robot description, xacro)
@@ -1,4 +1,4 @@
 <?xml version="1.0"?>
-<robot xmlns:xacro="http://wiki.ros.org/xacro" name="$(arg name)">
+<robot xmlns:xacro="http://wiki.ros.org/xacro" name="ur10">
   <xacro:arg name="name" default="ur10"/>
   <xacro:arg name="tf_prefix" default=""/>
