Commit message: gripper close and open working with moveit

File: ros2_ws/src/robotiq_3f_gripper_description/urdf/robotiq_3f_finger_macro.xacro (robot description, xacro)
@@ -7,8 +7,8 @@
 -->
 <robot xmlns:xacro="http://ros.org/wiki/xacro">
-  <xacro:macro name="robotiq_3f_finger_articulated" params="prefix axis_sign=1">
+  <xacro:macro name="robotiq_3f_finger_articulated" params="prefix axis_sign=1 face_flip=0">
     <link name="${prefix}link_0">
       <visual>
-        <origin xyz="0.020 0 0" rpy="0 0 0"/>
+        <origin xyz="0.020 0 0" rpy="${face_flip*3.1416} 0 0"/>
         <geometry>
           <mesh filename="package://robotiq_3f_gripper_description/meshes/visual/link_0.dae"/>
@@ -19,5 +19,5 @@
       </visual>
       <collision>
-        <origin xyz="0.020 0 0" rpy="0 0 0"/>
+        <origin xyz="0.020 0 0" rpy="${face_flip*3.1416} 0 0"/>
         <geometry>
           <mesh filename="package://robotiq_3f_gripper_description/meshes/collision/link_0.STL"/>
@@ -32,5 +32,5 @@
     <link name="${prefix}link_1">
       <visual>
-        <origin xyz="0.050 -0.028 0" rpy="0 0 -0.52"/>
+        <origin xyz="0.050 -0.028 0" rpy="${face_flip*3.1416} 0 -0.52"/>
         <geometry>
           <mesh filename="package://robotiq_3f_gripper_description/meshes/visual/link_1.dae"/>
@@ -41,5 +41,5 @@
       </visual>
       <collision>
-        <origin xyz="0.050 -0.028 0" rpy="0 0 -0.52"/>
+        <origin xyz="0.050 -0.028 0" rpy="${face_flip*3.1416} 0 -0.52"/>
         <geometry>
           <mesh filename="package://robotiq_3f_gripper_description/meshes/collision/link_1.STL"/>
@@ -54,5 +54,5 @@
     <link name="${prefix}link_2">
       <visual>
-        <origin xyz="0.039 0 0.0075" rpy="0 0 0"/>
+        <origin xyz="0.039 0 0.0075" rpy="${face_flip*3.1416} 0 0"/>
         <geometry>
           <mesh filename="package://robotiq_3f_gripper_description/meshes/visual/link_2.dae"/>
@@ -61,5 +61,5 @@
       </visual>
       <collision>
-        <origin xyz="0.039 0 0.0075" rpy="0 0 0"/>
+        <origin xyz="0.039 0 0.0075" rpy="${face_flip*3.1416} 0 0"/>
         <geometry>
           <mesh filename="package://robotiq_3f_gripper_description/meshes/collision/link_2.STL"/>
@@ -74,5 +74,5 @@
     <link name="${prefix}link_3">
       <visual>
-        <origin xyz="0 0 0" rpy="0 0 0.52"/>
+        <origin xyz="0 0 0" rpy="${face_flip*3.1416} 0 0.52"/>
         <geometry>
           <mesh filename="package://robotiq_3f_gripper_description/meshes/visual/link_3.dae"/>
@@ -81,5 +81,5 @@
       </visual>
       <collision>
-        <origin xyz="0 0 0" rpy="0 0 0.52"/>
+        <origin xyz="0 0 0" rpy="${face_flip*3.1416} 0 0.52"/>
         <geometry>
           <mesh filename="package://robotiq_3f_gripper_description/meshes/collision/link_3.STL"/>
@@ -113,108 +113,3 @@
     </joint>
   </xacro:macro>
-  <xacro:macro name="robotiq_3f_middle_finger_articulated" params="prefix">
-    <link name="${prefix}link_0">
-      <visual>
-        <origin xyz="0.020 0 0" rpy="0 0 0"/>
-        <geometry>
-          <mesh filename="package://robotiq_3f_gripper_description/meshes/visual/link_0.dae"/>
-        </geometry>
-        <material name="gripper_dark">
-          <color rgba="0.12 0.12 0.13 1"/>
-        </material>
-      </visual>
-      <collision>
-        <origin xyz="0.020 0 0" rpy="0 0 0"/>
-        <geometry>
-          <mesh filename="package://robotiq_3f_gripper_description/meshes/collision/link_0.STL"/>
-        </geometry>
-      </collision>
-      <inertial>
-          <origin xyz="0 0 0" rpy="0 0 0"/>
-          <mass value="0.05"/>
-          <inertia ixx="4.9e-6" ixy="0" ixz="0" iyy="9.1e-6" iyz="0" izz="9.1e-6" />
-      </inertial>
-    </link>
-    <link name="${prefix}link_1">
-      <visual>
-        <origin xyz="0.050 0.028 0" rpy="0 0 0.52"/>
-        <geometry>
-          <mesh filename="package://robotiq_3f_gripper_description/meshes/visual/link_1.dae"/>
-        </geometry>
-        <material name="gripper_light">
-          <color rgba="0.65 0.66 0.68 1"/>
-        </material>
-      </visual>
-      <collision>
-        <origin xyz="0.050 0.028 0" rpy="0 0 0.52"/>
-        <geometry>
-          <mesh filename="package://robotiq_3f_gripper_description/meshes/collision/link_1.STL"/>
-        </geometry>
-      </collision>
-      <inertial>
-          <origin xyz="0 0 0" rpy="0 0 0"/>
-          <mass value="0.15"/>
-          <inertia ixx="1.08e-5" ixy="0" ixz="0" iyy="6.67e-5" iyz="0" izz="6.67e-5" />
-      </inertial>
-    </link>
-    <link name="${prefix}link_2">
-      <visual>
-        <origin xyz="0.039 0 0.0075" rpy="0 0 0"/>
-        <geometry>
-          <mesh filename="package://robotiq_3f_gripper_description/meshes/visual/link_2.dae"/>
-        </geometry>
-        <material name="gripper_light"/>
-      </visual>
-      <collision>
-        <origin xyz="0.039 0 0.0075" rpy="0 0 0"/>
-        <geometry>
-          <mesh filename="package://robotiq_3f_gripper_description/meshes/collision/link_2.STL"/>
-        </geometry>
-      </collision>
-      <inertial>
-          <origin xyz="0 0 0" rpy="0 0 0"/>
-          <mass value="0.05"/>
-          <inertia ixx="2.5e-6" ixy="0" ixz="0" iyy="7.9e-6" iyz="0" izz="7.9e-6" />
-      </inertial>
-    </link>
-    <link name="${prefix}link_3">
-      <visual>
-        <origin xyz="0 0 0" rpy="0 0 -0.52"/>
-        <geometry>
-          <mesh filename="package://robotiq_3f_gripper_description/meshes/visual/link_3.dae"/>
-        </geometry>
-        <material name="gripper_light"/>
-      </visual>
-      <collision>
-        <origin xyz="0 0 0" rpy="0 0 -0.52"/>
-        <geometry>
-          <mesh filename="package://robotiq_3f_gripper_description/meshes/collision/link_3.STL"/>
-        </geometry>
-      </collision>
-      <inertial>
-        <origin xyz="0 0 0" rpy="0 0 0"/>
-        <mass value="0.05"/>
-        <inertia ixx="0.001239" ixy="-0.000251" ixz="0.000019" iyy="0.00085" iyz="0" izz="0.001632"/>
-      </inertial>
-    </link>
-    <joint name="${prefix}joint_1" type="revolute">
-      <parent link="${prefix}link_0"/>
-      <child link="${prefix}link_1"/>
-      <!-- The middle finger is mounted on the opposite side of the palm, so it
-           needs the mirrored sign to keep the physical closing motion consistent. -->
-      <axis xyz="0 0 -1"/>
-      <origin xyz="0.020 0 0" rpy="0 0 0"/>
-      <limit lower="0.0495" upper="1.2218" effort="100" velocity="1.0"/>
-    </joint>
-    <joint name="${prefix}joint_2" type="fixed">
-      <parent link="${prefix}link_1"/>
-      <child link="${prefix}link_2"/>
-      <origin xyz="0.050 0.028 0" rpy="0 0 0.52"/>
-    </joint>
-    <joint name="${prefix}joint_3" type="fixed">
-      <parent link="${prefix}link_2"/>
-      <child link="${prefix}link_3"/>
-      <origin xyz="0.039 0 0" rpy="0 0 0"/>
-    </joint>
-  </xacro:macro>
 </robot>

File: ros2_ws/src/robotiq_3f_gripper_description/urdf/robotiq_3f_gripper_macro.xacro (robot description, xacro)
@@ -53,5 +53,5 @@
     <xacro:robotiq_3f_finger_articulated prefix="${prefix}finger_1_" axis_sign="1"/>
     <xacro:robotiq_3f_finger_articulated prefix="${prefix}finger_2_" axis_sign="1"/>
-    <xacro:robotiq_3f_middle_finger_articulated prefix="${prefix}finger_middle_"/>
+    <xacro:robotiq_3f_finger_articulated prefix="${prefix}finger_middle_" axis_sign="-1" face_flip="-1"/>
     <joint name="${prefix}palm_finger_1_joint" type="fixed">
       <parent link="${prefix}palm"/>
@@ -67,8 +67,6 @@
       <parent link="${prefix}palm"/>
       <child link="${prefix}finger_middle_link_0"/>
-      <!-- The middle finger sits on the opposite side of the palm and needs the
-           same mirror/pitch adjustment that the original Robotiq geometry used,
-           while the mirrored joint sign keeps the command convention consistent. -->
-      <origin xyz="0.0455 0.0214 0" rpy="0 3.1416 1.57"/>
+      <!-- Keep the middle finger in the original Robotiq in-plane orientation. -->
+      <origin xyz="0.0455 0.0214 0" rpy="0 3.1416 -1.57"/>
     </joint>
   </xacro:macro>
