Commit message: gripper moveit working, except for third finger

File: ros2_ws/src/robotiq_3f_gripper_description/urdf/robotiq_3f_gripper_macro.xacro (robot description, xacro)
@@ -37,5 +37,9 @@
         <origin xyz="0 0 0" rpy="0 0 0"/>
         <mass value="1.3"/>
-        <inertia ixx="0.006012" ixy="0.000079" ixz="-0.00024" iyy="0.012892" iyz="0" izz="0.002435"/>
+        <!-- box approximation (~0.09 x 0.09 x 0.06 m), triangle-inequality-valid.
+             Original Robotiq spec values (ixx=0.006012, ixy=0.000079, ixz=-0.00024,
+             iyy=0.012892, izz=0.002435) fail ixx+izz >= iyy and are rejected by
+             SDFormat once lumped with the finger_middle branch. -->
+        <inertia ixx="0.0012675" ixy="0" ixz="0" iyy="0.0012675" iyz="0" izz="0.001755"/>
       </inertial>
     </link>
@@ -60,5 +64,5 @@
       <origin xyz="-0.0455 0.0214 -0.036" rpy="0 3.1416 -1.57"/>
     </joint>
-    <joint name="${prefix}palm_finger_middle_joint" type="fixed">
+        <joint name="${prefix}palm_finger_middle_joint" type="fixed">
       <parent link="${prefix}palm"/>
       <child link="${prefix}finger_middle_link_0"/>

Commit message: Implement collision checking for gripper states and update URDF/SRDF configurations for collision handling

File: ros2_ws/src/robotiq_3f_gripper_description/urdf/robotiq_3f_gripper_macro.xacro (robot description, xacro)
@@ -54,4 +54,19 @@
     <xacro:robotiq_3f_finger_articulated prefix="${prefix}finger_2_"/>
     <xacro:robotiq_3f_finger_articulated prefix="${prefix}finger_middle_"/>
+    <gazebo reference="${prefix}palm">
+      <selfCollide>false</selfCollide>
+    </gazebo>
+    <gazebo reference="${prefix}finger_middle_link_0">
+      <selfCollide>false</selfCollide>
+    </gazebo>
+    <gazebo reference="${prefix}finger_middle_link_1">
+      <selfCollide>false</selfCollide>
+    </gazebo>
+    <gazebo reference="${prefix}finger_middle_link_2">
+      <selfCollide>false</selfCollide>
+    </gazebo>
+    <gazebo reference="${prefix}finger_middle_link_3">
+      <selfCollide>false</selfCollide>
+    </gazebo>
     <joint name="${prefix}palm_finger_1_joint" type="fixed">
       <parent link="${prefix}palm"/>
@@ -64,5 +79,5 @@
       <origin xyz="-0.0455 0.0214 -0.036" rpy="0 3.1416 -1.57"/>
     </joint>
-        <joint name="${prefix}palm_finger_middle_joint" type="fixed">
+    <joint name="${prefix}palm_finger_middle_joint" type="fixed">
       <parent link="${prefix}palm"/>
       <child link="${prefix}finger_middle_link_0"/>

Commit message: Enhance UR10 control and gripper integration: update build command, adjust gripper joint positions, add gripper sequence node, refine MoveIt configuration, and clean up RViz settings.

File: ros2_ws/src/robotiq_3f_gripper_description/urdf/robotiq_3f_gripper_macro.xacro (robot description, xacro)
@@ -68,5 +68,5 @@
       <child link="${prefix}finger_middle_link_0"/>
       <!-- Keep the middle finger in the original Robotiq in-plane orientation. -->
-      <origin xyz="0.0455 0.0214 0" rpy="0 3.1416 -1.57"/>
+      <origin xyz="0.0580 0.0214 0" rpy="0 3.1416 -1.95"/>
     </joint>
   </xacro:macro>
