Commit message: Add camera alignment functionality and update world configuration for simulation

File: ros2_ws/src/vendor/robotiq_3f_gripper_description/urdf/ur10_robotiq_3f.urdf.xacro (robot description, xacro)
@@ -12,3 +12,60 @@
   </xacro:robotiq_3f_gripper_articulated>
   <xacro:robotiq_3f_gripper_ros2_control prefix="$(arg gripper_prefix)" sim_ignition="$(arg sim_ignition)"/>
+  <!-- ===================== Wrist-mounted RGBD camera ===================== -->
+  <link name="wrist_camera_link">
+    <visual>
+      <origin xyz="0 0 0" rpy="0 0 0"/>
+      <geometry>
+        <box size="0.02 0.05 0.02"/>
+      </geometry>
+      <material name="camera_body">
+        <color rgba="0.75 0.75 0.75 1"/>
+      </material>
+    </visual>
+    <visual>
+      <!-- Lens marker: small dark nub offset along local +Y, matching where
+          the sensor's forward pose actually points after the pitch rotation -->
+      <origin xyz="0 0.03 0" rpy="0 0 0"/>
+      <geometry>
+        <box size="0.012 0.012 0.012"/>
+      </geometry>
+      <material name="camera_lens">
+        <color rgba="0.05 0.05 0.05 1"/>
+      </material>
+    </visual>
+  </link>
+  <joint name="wrist_camera_joint" type="fixed">
+    <parent link="tool0"/>
+    <child link="wrist_camera_link"/>
+    <origin rpy="0 0 1.5708" xyz="0.0 -0.07 0.0"/>
+  </joint>
+  <!-- Optical frame: Gazebo sensor convention (Z-forward) differs from the
+      mechanical link (X-forward), ROS image pipelines expect the optical
+      frame's orientation, not the mechanical one -->
+  <link name="wrist_camera_link_optical"/>
+  <joint name="wrist_camera_optical_joint" type="fixed">
+    <parent link="wrist_camera_link"/>
+    <child link="wrist_camera_link_optical"/>
+    <origin xyz="0 0 0" rpy="-1.5708 0 -1.5708"/>
+  </joint>
+  <gazebo reference="wrist_camera_link">
+    <sensor name="wrist_rgbd_camera" type="rgbd_camera">
+      <pose>0 0 0 0 1.5708 0</pose>
+      <always_on>true</always_on>
+      <update_rate>15</update_rate>
+      <topic>wrist_camera</topic>
+      <camera>
+        <horizontal_fov>1.047</horizontal_fov>
+        <image>
+          <width>640</width>
+          <height>480</height>
+        </image>
+        <clip>
+          <near>0.05</near>
+          <far>3.0</far>
+        </clip>
+        <optical_frame_id>wrist_camera_link_optical</optical_frame_id>
+      </camera>
+    </sensor>
+  </gazebo>
 </robot>

Commit message: added still camera with point cloud and depth image feed

File: ros2_ws/src/vendor/robotiq_3f_gripper_description/urdf/ur10_robotiq_3f.urdf.xacro (robot description, xacro)
@@ -12,60 +12,3 @@
   </xacro:robotiq_3f_gripper_articulated>
   <xacro:robotiq_3f_gripper_ros2_control prefix="$(arg gripper_prefix)" sim_ignition="$(arg sim_ignition)"/>
-  <!-- ===================== Wrist-mounted RGBD camera ===================== -->
-  <link name="wrist_camera_link">
-    <visual>
-      <origin xyz="0 0 0" rpy="0 0 0"/>
-      <geometry>
-        <box size="0.02 0.05 0.02"/>
-      </geometry>
-      <material name="camera_body">
-        <color rgba="0.75 0.75 0.75 1"/>
-      </material>
-    </visual>
-    <visual>
-      <!-- Lens marker: small dark nub offset along local +Y, matching where
-          the sensor's forward pose actually points after the pitch rotation -->
-      <origin xyz="0 0.03 0" rpy="0 0 0"/>
-      <geometry>
-        <box size="0.012 0.012 0.012"/>
-      </geometry>
-      <material name="camera_lens">
-        <color rgba="0.05 0.05 0.05 1"/>
-      </material>
-    </visual>
-  </link>
-  <joint name="wrist_camera_joint" type="fixed">
-    <parent link="tool0"/>
-    <child link="wrist_camera_link"/>
-    <origin rpy="0 0 1.5708" xyz="0.0 -0.07 0.0"/>
-  </joint>
-  <!-- Optical frame: Gazebo sensor convention (Z-forward) differs from the
-      mechanical link (X-forward), ROS image pipelines expect the optical
-      frame's orientation, not the mechanical one -->
-  <link name="wrist_camera_link_optical"/>
-  <joint name="wrist_camera_optical_joint" type="fixed">
-    <parent link="wrist_camera_link"/>
-    <child link="wrist_camera_link_optical"/>
-    <origin xyz="0 0 0" rpy="-1.5708 0 -1.5708"/>
-  </joint>
-  <gazebo reference="wrist_camera_link">
-    <sensor name="wrist_rgbd_camera" type="rgbd_camera">
-      <pose>0 0 0 0 1.5708 0</pose>
-      <always_on>true</always_on>
-      <update_rate>15</update_rate>
-      <topic>wrist_camera</topic>
-      <camera>
-        <horizontal_fov>1.047</horizontal_fov>
-        <image>
-          <width>640</width>
-          <height>480</height>
-        </image>
-        <clip>
-          <near>0.05</near>
-          <far>3.0</far>
-        </clip>
-        <optical_frame_id>wrist_camera_link_optical</optical_frame_id>
-      </camera>
-    </sensor>
-  </gazebo>
 </robot>

Commit message: point cloud for real hardware fixed, offset in z axis fixed due to missing sensor joint in sim, real grasp and pick not yet error free

File: ros2_ws/src/vendor/robotiq_3f_gripper_description/urdf/ur10_robotiq_3f.urdf.xacro (robot description, xacro)
@@ -5,9 +5,10 @@
   <xacro:arg name="gripper_prefix" default="gripper_"/>
   <xacro:arg name="sim_ignition" default="true"/>
+  <xacro:arg name="sensor_mount_offset" default="0.081"/>
   <xacro:include filename="$(find ur_description)/urdf/ur.urdf.xacro"/>
   <xacro:include filename="$(find robotiq_3f_gripper_description)/urdf/robotiq_3f_gripper_macro.xacro"/>
   <xacro:include filename="$(find robotiq_3f_gripper_description)/urdf/robotiq_3f_gripper_ros2_control.xacro"/>
   <xacro:robotiq_3f_gripper_articulated prefix="$(arg gripper_prefix)" parent="$(arg tf_prefix)tool0">
-    <origin xyz="0 0 0" rpy="1.5708 0 0"/>
+    <origin xyz="0 0 $(arg sensor_mount_offset)" rpy="1.5708 0 0"/>
   </xacro:robotiq_3f_gripper_articulated>
   <xacro:robotiq_3f_gripper_ros2_control prefix="$(arg gripper_prefix)" sim_ignition="$(arg sim_ignition)"/>
