Commit message: gripper issue solved and mounted properly

File: ros2_ws/src/vendor/robotiq_3f_gripper_description/urdf/robotiq_3f_finger_macro.xacro (robot description, xacro)
@@ -7,5 +7,5 @@
 -->
 <robot xmlns:xacro="http://ros.org/wiki/xacro">
-  <xacro:macro name="robotiq_3f_finger_articulated" params="prefix axis_sign=1 face_flip=0">
+  <xacro:macro name="robotiq_3f_finger_articulated" params="prefix axis_sign=1 face_flip=0 articulated=false">
     <link name="${prefix}link_0">
       <visual>
@@ -100,16 +100,32 @@
       <axis xyz="0 0 ${axis_sign}"/>
       <origin xyz="0.020 0 0" rpy="0 0 0"/>
-      <limit lower="0.0495" upper="1.2218" effort="100" velocity="1.0"/>
+      <limit lower="0.0445" upper="1.2718" effort="100" velocity="1.0"/>
     </joint>
+    <xacro:if value="${articulated}">
+    <joint name="${prefix}joint_2" type="revolute">
+      <parent link="${prefix}link_1"/><child link="${prefix}link_2"/>
+      <axis xyz="0 0 ${axis_sign}"/>
+      <origin xyz="0.050 -0.028 0" rpy="0 0 -0.52"/>
+      <limit lower="0.0" upper="1.6472" effort="100" velocity="100"/>
+      <mimic joint="${prefix}joint_1" multiplier="1.3400" offset="-0.0663"/>
+    </joint>
+    <joint name="${prefix}joint_3" type="revolute">
+      <parent link="${prefix}link_2"/><child link="${prefix}link_3"/>
+      <axis xyz="0 0 ${axis_sign}"/>
+      <origin xyz="0.039 0 0" rpy="0 0 0"/>
+      <limit lower="-1.2217" upper="-0.0400" effort="100" velocity="100"/>
+      <mimic joint="${prefix}joint_1" multiplier="-0.9975" offset="-0.0029"/>
+    </joint>
+  </xacro:if>
+  <xacro:unless value="${articulated}">
     <joint name="${prefix}joint_2" type="fixed">
-      <parent link="${prefix}link_1"/>
-      <child link="${prefix}link_2"/>
+      <parent link="${prefix}link_1"/><child link="${prefix}link_2"/>
       <origin xyz="0.050 -0.028 0" rpy="0 0 -0.52"/>
     </joint>
     <joint name="${prefix}joint_3" type="fixed">
-      <parent link="${prefix}link_2"/>
-      <child link="${prefix}link_3"/>
+      <parent link="${prefix}link_2"/><child link="${prefix}link_3"/>
       <origin xyz="0.039 0 0" rpy="0 0 0"/>
     </joint>
+  </xacro:unless>
   </xacro:macro>
 </robot>

File: ros2_ws/src/vendor/robotiq_3f_gripper_description/urdf/robotiq_3f_gripper_macro.xacro (robot description, xacro)
@@ -14,5 +14,5 @@
 <robot xmlns:xacro="http://ros.org/wiki/xacro">
   <xacro:include filename="$(find robotiq_3f_gripper_description)/urdf/robotiq_3f_finger_macro.xacro"/>
-  <xacro:macro name="robotiq_3f_gripper_articulated" params="prefix parent *origin">
+  <xacro:macro name="robotiq_3f_gripper_articulated" params="prefix parent *origin articulated:=false" >
     <joint name="${prefix}palm_joint" type="fixed">
       <parent link="${parent}"/>
@@ -51,7 +51,7 @@
       <origin xyz="0.0 0.0875 0.0" rpy="0 0 1.5707"/>
     </joint>
-    <xacro:robotiq_3f_finger_articulated prefix="${prefix}finger_1_" axis_sign="1"/>
-    <xacro:robotiq_3f_finger_articulated prefix="${prefix}finger_2_" axis_sign="1"/>
-    <xacro:robotiq_3f_finger_articulated prefix="${prefix}finger_middle_" axis_sign="-1" face_flip="-1"/>
+    <xacro:robotiq_3f_finger_articulated prefix="${prefix}finger_1_" axis_sign="1" articulated="${articulated}"/>
+    <xacro:robotiq_3f_finger_articulated prefix="${prefix}finger_2_" axis_sign="1" articulated="${articulated}"/>
+    <xacro:robotiq_3f_finger_articulated prefix="${prefix}finger_middle_" articulated="${articulated}"/>
     <joint name="${prefix}palm_finger_1_joint" type="fixed">
       <parent link="${prefix}palm"/>
@@ -68,5 +68,5 @@
       <child link="${prefix}finger_middle_link_0"/>
       <!-- Keep the middle finger in the original Robotiq in-plane orientation. -->
-      <origin xyz="0.0580 0.0214 0" rpy="0 3.1416 -1.95"/>
+      <origin xyz="0.0455 0.0114 0" rpy="0 0 1.1916"/>
     </joint>
   </xacro:macro>

File: ros2_ws/src/vendor/robotiq_3f_gripper_description/urdf/robotiq_3f_gripper_ros2_control.xacro (robot description, xacro)
@@ -1,7 +1,19 @@
 <?xml version="1.0"?>
 <robot xmlns:xacro="http://ros.org/wiki/xacro">
+  <xacro:macro name="robotiq_3f_finger_mimic" params="prefix finger">
+    <joint name="${prefix}${finger}joint_2">
+      <param name="mimic">${prefix}${finger}joint_1</param>
+      <param name="multiplier">1.3400</param>
+      <state_interface name="position"/>
+    </joint>
+    <joint name="${prefix}${finger}joint_3">
+      <param name="mimic">${prefix}${finger}joint_1</param>
+      <param name="multiplier">-0.9975</param>
+      <state_interface name="position"/>
+    </joint>
+  </xacro:macro>
   <xacro:macro
     name="robotiq_3f_gripper_ros2_control"
-    params="prefix sim_ignition:=true">
+    params="prefix sim_ignition:=true articulated:=false">
     <ros2_control name="${prefix}gripper_system" type="system">
       <hardware>
@@ -43,4 +55,9 @@
         <state_interface name="velocity"/>
       </joint>
+      <xacro:if value="${articulated}">
+        <xacro:robotiq_3f_finger_mimic prefix="${prefix}" finger="finger_1_"/>
+        <xacro:robotiq_3f_finger_mimic prefix="${prefix}" finger="finger_2_"/>
+        <xacro:robotiq_3f_finger_mimic prefix="${prefix}" finger="finger_middle_"/>
+      </xacro:if>
     </ros2_control>
   </xacro:macro>

File: ros2_ws/src/vendor/robotiq_3f_gripper_description/urdf/ur10_robotiq_3f.urdf.xacro (robot description, xacro)
@@ -6,10 +6,39 @@
   <xacro:arg name="sim_ignition" default="true"/>
   <xacro:arg name="sensor_mount_offset" default="0.081"/>
+  <xacro:arg name="articulated_fingers" default="false"/>
   <xacro:include filename="$(find ur_description)/urdf/ur.urdf.xacro"/>
   <xacro:include filename="$(find robotiq_3f_gripper_description)/urdf/robotiq_3f_gripper_macro.xacro"/>
   <xacro:include filename="$(find robotiq_3f_gripper_description)/urdf/robotiq_3f_gripper_ros2_control.xacro"/>
-  <xacro:robotiq_3f_gripper_articulated prefix="$(arg gripper_prefix)" parent="$(arg tf_prefix)tool0">
+  <xacro:robotiq_3f_gripper_articulated prefix="$(arg gripper_prefix)" parent="$(arg tf_prefix)tool0" articulated="$(arg articulated_fingers)">
     <origin xyz="0 0 $(arg sensor_mount_offset)" rpy="1.5708 0 0"/>
   </xacro:robotiq_3f_gripper_articulated>
-  <xacro:robotiq_3f_gripper_ros2_control prefix="$(arg gripper_prefix)" sim_ignition="$(arg sim_ignition)"/>
+  <xacro:arg name="sensor_mount_radius" default="0.035"/>
+  <xacro:arg name="sensor_mount_mass" default="0.3"/>
+  <xacro:property name="sensor_mount_len" value="$(arg sensor_mount_offset)"/>
+  <xacro:property name="sensor_mount_r" value="$(arg sensor_mount_radius)"/>
+  <xacro:property name="sensor_mount_m" value="$(arg sensor_mount_mass)"/>
+  <link name="$(arg gripper_prefix)sensor_mount">
+    <visual>
+      <origin xyz="0 0 ${sensor_mount_len/2}" rpy="0 0 0"/>
+      <geometry><cylinder radius="${sensor_mount_r}" length="${sensor_mount_len}"/></geometry>
+      <material name="sensor_mount"><color rgba="0.3 0.3 0.32 1"/></material>
+    </visual>
+    <collision>
+      <origin xyz="0 0 ${sensor_mount_len/2}" rpy="0 0 0"/>
+      <geometry><cylinder radius="${sensor_mount_r}" length="${sensor_mount_len}"/></geometry>
+    </collision>
+    <inertial>
+      <origin xyz="0 0 ${sensor_mount_len/2}" rpy="0 0 0"/>
+      <mass value="${sensor_mount_m}"/>
+      <inertia ixx="${sensor_mount_m*(3*sensor_mount_r*sensor_mount_r+sensor_mount_len*sensor_mount_len)/12}" ixy="0" ixz="0"
+               iyy="${sensor_mount_m*(3*sensor_mount_r*sensor_mount_r+sensor_mount_len*sensor_mount_len)/12}" iyz="0"
+               izz="${sensor_mount_m*sensor_mount_r*sensor_mount_r/2}"/>
+    </inertial>
+  </link>
+  <joint name="$(arg gripper_prefix)sensor_mount_joint" type="fixed">
+    <parent link="$(arg tf_prefix)tool0"/>
+    <child link="$(arg gripper_prefix)sensor_mount"/>
+    <origin xyz="0 0 0" rpy="0 0 0"/>
+  </joint>
+  <xacro:robotiq_3f_gripper_ros2_control prefix="$(arg gripper_prefix)" sim_ignition="$(arg sim_ignition)" articulated="$(arg articulated_fingers)"/>
 </robot>
